Commit message: rearranged charger in urdf model

File: urdf/vmecanumrover.xacro (robot description, xacro)
@@ -1,4 +1,13 @@
 <?xml version="1.0"?>
 <robot name="vmecanumrover" xmlns:xacro="http://ros.org/wiki/xacro">
+   <material name="black">
+    <color rgba="0.0 0.0 0.0 1.0"/>
+  </material>
+  <material name="gray">
+    <color rgba="0.7 0.7 0.7 1.0"/>
+  </material>
+  <material name="red">
+    <color rgba="0.8 0.0 0.0 1.0"/>
+  </material>
   <link name="base_link"/>
   <xacro:macro name="cylinder_inertial" params="mass radius length">
@@ -419,6 +428,6 @@
     <sensor type="ray" name="lidar_sensor">
       <pose>0 0 0 0 0 0</pose>
-      <visualize>true</visualize>
-      <update_rate>40</update_rate>
+      <visualize>false</visualize>
+      <update_rate>20</update_rate>
       <ray>
         <scan>
@@ -432,5 +441,5 @@
         <range>
           <min>0.06</min>
-          <max>4.0</max>
+          <max>14.0</max>
         <resolution>0.001</resolution>
         </range>
@@ -474,7 +483,6 @@
   <!-- Wyreless charger  -->
   <!-- attachiment  -->
-<!--
   <joint name="charger_attach_joint" type="fixed">
-    <parent link="board_front_link"/>
+    <parent link="board_back_link"/>
     <child  link="charger_attach_link"/>
     <origin xyz="0.06 0 -0.0015" rpy="0 0 0"/>
@@ -499,7 +507,5 @@
     <material>Gazebo/White</material>
   </gazebo>
--->
   <!-- wyreless charger  -->
-<!--
   <joint name="charger_joint" type="prismatic">
     <parent link="charger_attach_link"/>
@@ -544,5 +550,4 @@
     <kd value="100" />
   </gazebo>
--->
   <!-- NUC PC  -->
   <!-- option attach board  -->

Commit message: updated teb params, added slam toolbox mapping, added prerequisites for ekf

File: urdf/vmecanumrover.xacro (robot description, xacro)
@@ -601,4 +601,39 @@
     <material>Gazebo/Black</material>
   </gazebo>
+  <joint name="imu_joint" type="fixed">
+    <parent link="base_link"/>
+    <child link="imu_link"/>
+    <origin xyz="0 0 0" rpy="0 0 0"/>
+  </joint>
+  <link name="imu_link"/>
+  <gazebo>
+    <plugin name="imu_plugin" filename="libgazebo_ros_imu.so">
+      <alwaysOn>true</alwaysOn>
+      <bodyName>imu_link</bodyName>
+      <frameName>imu_link</frameName>
+      <topicName>imu</topicName>
+      <serviceName>imu_service</serviceName>
+      <gaussianNoise>0.0</gaussianNoise>
+      <updateRate>100</updateRate>
+      <imu>
+        <noise>
+          <type>gaussian</type>
+          <rate>
+            <mean>0.0</mean>
+            <stddev>2e-4</stddev>
+            <bias_mean>0.0000075</bias_mean>
+            <bias_stddev>0.0000008</bias_stddev>
+          </rate>
+          <accel>
+            <mean>0.0</mean>
+            <stddev>1.7e-2</stddev>
+            <bias_mean>0.1</bias_mean>
+            <bias_stddev>0.001</bias_stddev>
+          </accel>
+        </noise>
+      </imu>
+      <robotNamespace>/vmecanumrover</robotNamespace>
+    </plugin>
+  </gazebo>
   <gazebo>
     <plugin name="gazebo_ros_control" filename="libgazebo_ros_control.so">
